Commit message: updated

File: install/rover_description/share/rover_description/robots/rover.urdf.xacro (robot description, xacro)
@@ -30,10 +30,9 @@
     <xacro:include filename="$(find rover_description)/urdf/wheels/corner.urdf.xacro" />
     <xacro:include filename="$(find rover_description)/urdf/sensors/all_sensors.urdf.xacro" />
-    <gazebo>
+        <gazebo>
         <plugin filename="gz_ros2_control-system" name="gz_ros2_control::GazeboSimROS2ControlPlugin">
             <parameters>$(find rover_description)/config/control.yaml</parameters>
             <ros>
-                <remapping>/tf:=tf</remapping>
-                <remapping>/tf_static:=tf_static</remapping>
+                <namespace>/</namespace>
             </ros>
         </plugin>

File: install/rover_description/share/rover_description/urdf/sensors/hokuyo.urdf.xacro (robot description, xacro)
@@ -18,9 +18,38 @@
 # SOFTWARE. -->
 <robot xmlns:xacro="http://www.ros.org/wiki/xacro">
-  <xacro:macro name="sensor_hokuyo" params="prefix parent *origin min_angle:=-3.14159265359 max_angle:=3.14159265359">
+  <xacro:macro name="sensor_hokuyo" params="prefix parent *origin min_angle:=-1.57079637051 max_angle:=1.57079637051">
     <joint name="${prefix}_base_joint" type="fixed">
       <xacro:insert_block name="origin" />
       <parent link="${parent}"/>
       <child link="${prefix}_base_link"/>
+    </joint>
+    <link name="${prefix}_base_link">
+      <collision>
+        <origin xyz="0 0 -0.05" rpy="0 0 0"/>
+        <geometry>
+          <box size="0.010 0.010 0.010"/>
+        </geometry>
+      </collision>
+      <visual>
+        <origin xyz="0 0 -0.05" rpy="0 0 0"/>
+        <geometry>
+          <mesh filename="package://rover_description/meshes/sensors/hokuyo/hokuyo_ust_20lx.dae"/>
+        </geometry>
+      </visual>
+      <inertial>
+        <mass value="1e-5" />
+        <origin xyz="0 0 0" rpy="0 0 0"/>
+        <inertia ixx="1e-6" ixy="0" ixz="0" iyy="1e-6" iyz="0" izz="1e-6" />
+      </inertial>
+    </link>
+    <gazebo reference="${prefix}_base_link">
+      <material>Gazebo/DarkGrey</material>
+    </gazebo>
+    <link name="${prefix}_link">
+    </link>
+    <joint name="${prefix}_joint" type="fixed">
+      <parent link="${prefix}_base_link"/>
+      <child link="${prefix}_link"/>
+      <origin xyz="0.00 0 0.0" rpy="0 0 0"/>
     </joint>
     <gazebo reference="${prefix}_link">
@@ -29,8 +58,9 @@
         <topic>/scan</topic>
         <update_rate>10</update_rate>
+        <gz_frame_id>${prefix}_link</gz_frame_id>
         <ray>
           <scan>
             <horizontal>
-              <samples>1081</samples>
+              <samples>360</samples>
               <resolution>1</resolution>
               <min_angle>${min_angle}</min_angle>

File: install/rover_description/share/rover_description/urdf/sensors/imu.urdf.xacro (robot description, xacro)
@@ -53,5 +53,5 @@
         <gz_frame_id>${prefix}_link</gz_frame_id>
         <always_on>1</always_on>
-        <update_rate>200</update_rate>
+        <update_rate>50</update_rate>
         <visualize>true</visualize>
         <pose relative_to="${prefix}_link">0 0 0 0 0 0</pose>
